Commit message: Phase 3b: TCP, dynamic cubes, KDL IK/FK services, grasp state machine

File: src/arm_description/urdf/arm.urdf.xacro (robot description, xacro)
@@ -155,5 +155,5 @@
     </inertial>
   </link>
-  <!-- joint 5: wrist pitch -->
+  <!-- joint 5: wrist pitch（±3.1 才能让夹爪朝下抓取） -->
   <joint name="joint5" type="revolute">
     <parent link="link4"/>
@@ -161,5 +161,5 @@
     <origin xyz="0 0 0.06" rpy="0 0 0"/>
     <axis xyz="0 1 0"/>
-    <limit lower="-2.0" upper="2.0" effort="10.0" velocity="2.0"/>
+    <limit lower="-3.1" upper="3.1" effort="10.0" velocity="2.0"/>
     <dynamics damping="0.1" friction="0.02"/>
   </joint>
@@ -223,5 +223,5 @@
       <origin xyz="0 0 0.015" rpy="0 0 0"/>
       <geometry>
-        <box size="0.09 0.07 0.03"/>
+        <box size="0.09 0.10 0.03"/>
       </geometry>
       <material name="rubber"/>
@@ -230,5 +230,5 @@
       <origin xyz="0 0 0.015" rpy="0 0 0"/>
       <geometry>
-        <box size="0.09 0.07 0.03"/>
+        <box size="0.09 0.10 0.03"/>
       </geometry>
     </collision>
@@ -239,9 +239,9 @@
     </inertial>
   </link>
-  <!-- left finger -->
+  <!-- left finger：闭合时间隙 40 mm，张开 15 mm 时间隙 70 mm，可夹 50 mm 方块 -->
   <joint name="finger_left_joint" type="prismatic">
     <parent link="gripper_base"/>
     <child link="finger_left"/>
-    <origin xyz="0 0.02 0" rpy="0 0 0"/>
+    <origin xyz="0 0.026 0" rpy="0 0 0"/>
     <axis xyz="0 1 0"/>
     <limit lower="0.0" upper="0.03" effort="10.0" velocity="0.05"/>
@@ -271,5 +271,5 @@
     <parent link="gripper_base"/>
     <child link="finger_right"/>
-    <origin xyz="0 -0.02 0" rpy="0 0 0"/>
+    <origin xyz="0 -0.026 0" rpy="0 0 0"/>
     <axis xyz="0 -1 0"/>
     <limit lower="0.0" upper="0.03" effort="10.0" velocity="0.05"/>
@@ -295,4 +295,25 @@
     </inertial>
   </link>
+  <!-- TCP：两指中点，位于夹爪基座下方 35 mm；抓取时对准方块中心 -->
+  <joint name="tcp_joint" type="fixed">
+    <parent link="gripper_base"/>
+    <child link="tcp"/>
+    <origin xyz="0 0 -0.035" rpy="0 0 0"/>
+  </joint>
+  <link name="tcp">
+    <inertial>
+      <mass value="0.01"/>
+      <inertia ixx="0.000001" ixy="0" ixz="0" iyy="0.000001" iyz="0" izz="0.000001"/>
+    </inertial>
+  </link>
+  <!-- 指垫摩擦：摩擦不足会导致抬升时方块滑落 -->
+  <gazebo reference="finger_left">
+    <mu1>5.0</mu1>
+    <mu2>5.0</mu2>
+  </gazebo>
+  <gazebo reference="finger_right">
+    <mu1>5.0</mu1>
+    <mu2>5.0</mu2>
+  </gazebo>
   <ros2_control name="GazeboSimSystem" type="system">
     <hardware>

Commit message: Phase 3b acceptance: grasp all three cubes, re-benchmark IK
Three chained root causes made descend abort with action status 6:
the IK target orientation was flipped 180 deg about x, the 5 mm tool
offset let the wrist barrel reach the cube, and grasp_height 0.032 put
that barrel 8 mm inside the 50 mm cube top face.

- grasp_node: identity+yaw grasp orientation, gripper_mount z -0.03
  (TCP 65 mm below tool0), grasp_height 0.050 with upward-only fallback
- kinematics_node: call CartToJnt, not JntToCart
- arm.urdf.xacro: joint3 effort 30 -> 100 (measured 37.8 N*m)
- launch: spawn controllers after the arm exists, longer spawner
  timeouts; bridge /model/cube_*/pose instead of world pose/info
- ik_benchmark: sample the orientation the grasp node actually uses,
  cube height 0.050

Measured on one clean launch: red/green/blue lifted 130/128/117 mm,
IK 28/30 = 93.3%, zero-pose FK 0.785 m, perception XY error 1-9 mm.
The previously reported 96.7% was measured at the flipped orientation
and is void.

File: src/arm_description/urdf/arm.urdf.xacro (robot description, xacro)
@@ -74,5 +74,5 @@
     <origin xyz="0 0 0.12" rpy="0 0 0"/>
     <axis xyz="0 1 0"/>
-    <limit lower="-2.0" upper="2.0" effort="30.0" velocity="1.5"/>
+    <limit lower="-2.0" upper="2.0" effort="100.0" velocity="1.5"/>
     <dynamics damping="0.2" friction="0.05"/>
   </joint>
@@ -103,5 +103,7 @@
     <origin xyz="0 0 0.30" rpy="0 0 0"/>
     <axis xyz="0 1 0"/>
-    <limit lower="-2.5" upper="2.5" effort="30.0" velocity="1.5"/>
+    <!-- effort 30 时远端目标（blue x≈0.48）descend 会被削顶，JTC 报 state tolerance；
+         gz_ros2_control 的位置 PID 起步索取力矩远大于重力矩（实测约 2 N·m），故与 joint2 同放到 100 -->
+    <limit lower="-2.5" upper="2.5" effort="100.0" velocity="1.5"/>
     <dynamics damping="0.2" friction="0.05"/>
   </joint>
@@ -213,9 +215,14 @@
     </inertial>
   </link>
-  <!-- gripper base -->
+  <!--
+    工具偏置：TCP +z 必须朝上，joint5/joint6 就得反向折约 127°，link5 的腕筒
+    被折到两指正中间、深到与指尖同高，下探时整个插进方块体积（指间净空 70 mm，
+    装不下腕筒 64 mm + 方块 50 mm）。夹爪整体下移 60 mm，TCP 落到 tool0 下方
+    65 mm，腕部才能留在物体上方。
+  -->
   <joint name="gripper_mount" type="fixed">
     <parent link="tool0"/>
     <child link="gripper_base"/>
-    <origin xyz="0 0 0.03" rpy="0 0 0"/>
+    <origin xyz="0 0 -0.03" rpy="0 0 0"/>
   </joint>
   <link name="gripper_base">
